Commit message: Add files via upload

File: simple_gripper.urdf (robot description, URDF)
Before this commit: robot simple_gripper, 6 links, 5 joints
Links:
- removed link left_finger
- removed link left_finger_tip
- removed link palm
- removed link right_finger
- removed link right_finger_tip
- removed link riser
- added link simple_gripper__left_finger, mass 0.1; collision box size=0.1 0.3 0.1; visual box size=0.1 0.3 0.1
- added link simple_gripper__left_finger_tip, mass 0.5; collision box size=0.1 0.2 0.1; visual box size=0.1 0.2 0.1
- added link simple_gripper__palm, mass 0.5; collision box size=0.1 0.2 0.1; visual box size=0.1 0.2 0.1
- added link simple_gripper__right_finger, mass 0.1; collision box size=0.1 0.3 0.1; visual box size=0.1 0.3 0.1
- added link simple_gripper__right_finger_tip, mass 0.1; collision box size=0.1 0.2 0.1; visual box size=0.1 0.2 0.1
- added link simple_gripper__riser, mass 10; collision box size=0.05 0.05 1.0; visual box size=0.05 0.05 1.0
Joints:
- removed joint left_finger_tip
- removed joint palm_left_finger
- removed joint palm_right_finger
- removed joint palm_riser
- removed joint right_finger_tip
- added joint simple_gripper__left_finger_tip: type revolute, parent simple_gripper__left_finger, child simple_gripper__left_finger_tip, origin xyz=0.02545 0.31688 0 rpy=0      0      2.35609, axis 0 0 1, limit lower=-0.8 upper=0.8 effort=0.0 velocity=0.0
- added joint simple_gripper__palm_left_finger: type revolute, parent simple_gripper__palm, child simple_gripper__left_finger, origin xyz=-0.00606  0.09393  0 rpy=0       0      -0.78539, axis 0 0 1, limit lower=-0.8 upper=0.8 effort=0.0 velocity=0.0
- added joint simple_gripper__palm_right_finger: type revolute, parent simple_gripper__palm, child simple_gripper__right_finger, origin xyz=-0.00606 -0.09393  0 rpy=0      0      0.78539, axis 0 0 1, limit lower=-0.8 upper=0.8 effort=0.0 velocity=0.0
- added joint simple_gripper__palm_riser: type prismatic, parent simple_gripper__riser, child simple_gripper__palm, origin xyz=0   0   0.05 rpy=0 0 0, axis 0 0 1, limit lower=0.0 upper=0.9 effort=0.0 velocity=0.0
- added joint simple_gripper__right_finger_tip: type revolute, parent simple_gripper__right_finger, child simple_gripper__right_finger_tip, origin xyz=0.02546 -0.31687  0 rpy=0      0      0.78531, axis 0 0 1, limit lower=-0.8 upper=0.8 effort=0.0 velocity=0.0

Commit message: Add files via upload
Added the third finger and its finger tip.

File: simple_gripper.urdf (robot description, URDF)
Before this commit: robot simple_gripper, 6 links, 5 joints
Links:
- added link simple_gripper__middle_finger, mass 0.1; collision box size=0.1 0.3 0.1; visual box size=0.1 0.1 0.3
- added link simple_gripper__middle_finger_tip, mass 0.1; collision box size=0.1 0.2 0.1; visual box size=0.1 0.1 0.2
- link simple_gripper__riser: mass 10 -> 3
Joints:
- added joint simple_gripper__middle_finger_tip: type revolute, parent simple_gripper__middle_finger, child simple_gripper__middle_finger_tip, origin xyz=0.02546 0 0.21687 rpy=0      0.78531     0, axis 0 1 0, limit lower=-0.8 upper=0.8 effort=0.0 velocity=0.0
- added joint simple_gripper__palm_middle_finger: type revolute, parent simple_gripper__palm, child simple_gripper__middle_finger, origin xyz=0 -0.00606 0.09393 rpy=0     0.78539    0, axis 0 1 0, limit lower=-0.8 upper=0.8 effort=0.0 velocity=0.0

Commit message: Add files via upload

File: simple_gripper.urdf (robot description, URDF)
Before this commit: robot simple_gripper, 8 links, 7 joints
Links:
- removed link simple_gripper__left_finger
- removed link simple_gripper__left_finger_tip
- removed link simple_gripper__middle_finger
- removed link simple_gripper__middle_finger_tip
- removed link simple_gripper__palm
- removed link simple_gripper__right_finger
- removed link simple_gripper__right_finger_tip
- removed link simple_gripper__riser
- added link left_finger, mass 0.1; collision box size=0.1 0.3 0.1; visual box size=0.1 0.3 0.1
- added link left_finger_tip, mass 0.5; collision box size=0.1 0.2 0.1; visual box size=0.1 0.2 0.1
- added link middle_finger, mass 0.1; collision box size=0.1 0.1 0.3; visual box size=0.1 0.1 0.3
- added link middle_finger_tip, mass 0.1; collision box size=0.1 0.1 0.2; visual box size=0.1 0.1 0.2
- added link palm, mass 0.5; collision box size=0.1 0.2 0.1; visual box size=0.1 0.2 0.1
- added link right_finger, mass 0.1; collision box size=0.1 0.3 0.1; visual box size=0.1 0.3 0.1
- added link right_finger_tip, mass 0.1; collision box size=0.1 0.2 0.1; visual box size=0.1 0.2 0.1
- added link riser, mass 3; collision box size=0.05 0.05 1.0; visual box size=0.05 0.05 1.0
Joints:
- removed joint simple_gripper__left_finger_tip
- removed joint simple_gripper__middle_finger_tip
- removed joint simple_gripper__palm_left_finger
- removed joint simple_gripper__palm_middle_finger
- removed joint simple_gripper__palm_right_finger
- removed joint simple_gripper__palm_riser
- removed joint simple_gripper__right_finger_tip
- added joint left_finger_tip: type revolute, parent left_finger, child left_finger_tip, origin xyz=0.02545 0.31688 0 rpy=0      0      2.35609, axis 0 0 1, limit lower=-0.8 upper=0.8 effort=0.0 velocity=0.0
- added joint middle_finger_tip: type revolute, parent middle_finger, child middle_finger_tip, origin xyz=0.02546 0 0.21687 rpy=0      0.78531     0, axis 0 1 0, limit lower=-0.8 upper=0.8 effort=0.0 velocity=0.0
- added joint palm_left_finger: type revolute, parent palm, child left_finger, origin xyz=-0.00606  0.09393  0 rpy=0       0      -0.78539, axis 0 0 1, limit lower=-0.8 upper=0.8 effort=0.0 velocity=0.0
- added joint palm_middle_finger: type revolute, parent palm, child middle_finger, origin xyz=0 -0.00606 0.09393 rpy=0     0.78539    0, axis 0 1 0, limit lower=-0.8 upper=0.670362 effort=0.0 velocity=0.0
- added joint palm_right_finger: type revolute, parent palm, child right_finger, origin xyz=-0.00606 -0.09393  0 rpy=0      0      0.78539, axis 0 0 1, limit lower=-0.8 upper=0.8 effort=0.0 velocity=0.0
- added joint palm_riser: type prismatic, parent riser, child palm, origin xyz=0   0   0.05 rpy=0 0 0, axis 0 0 1, limit lower=0.0 upper=0.9 effort=0.0 velocity=0.0
- added joint right_finger_tip: type revolute, parent right_finger, child right_finger_tip, origin xyz=0.02546 -0.31687  0 rpy=0      0      0.78531, axis 0 0 1, limit lower=-0.8 upper=0.8 effort=0.0 velocity=0.0

Commit message: Add files via upload

File: simple_gripper.urdf (robot description, URDF)
Before this commit: robot simple_gripper, 8 links, 7 joints
Links:
- added link world
Joints:
- added joint fixed: type fixed, parent world, child riser, origin xyz=0   0   -0.5 rpy=0 0 0
- joint left_finger_tip: limit lower=-0.8 upper=0.8 effort=0.0 velocity=0.0 -> lower=-0.8 upper=0.8 effort=1000.0 velocity=1000.0
- joint middle_finger_tip: limit lower=-0.8 upper=0.8 effort=0.0 velocity=0.0 -> lower=-0.8 upper=0.8 effort=1000.0 velocity=1000.0
- joint palm_left_finger: limit lower=-0.8 upper=0.8 effort=0.0 velocity=0.0 -> lower=-0.8 upper=0.8 effort=1000.0 velocity=1000.0
- joint palm_middle_finger: limit lower=-0.8 upper=0.670362 effort=0.0 velocity=0.0 -> lower=-0.8 upper=0.670362 effort=1000.0 velocity=1000.0
- joint palm_right_finger: limit lower=-0.8 upper=0.8 effort=0.0 velocity=0.0 -> lower=-0.8 upper=0.8 effort=1000.0 velocity=1000.0
- joint palm_riser: limit lower=0.0 upper=0.9 effort=0.0 velocity=0.0 -> lower=-0.5 upper=2 effort=1000.0 velocity=10.0; origin xyz=0   0   0.05 rpy=0 0 0 -> xyz=0   0   0 rpy=0 0 0
- joint right_finger_tip: limit lower=-0.8 upper=0.8 effort=0.0 velocity=0.0 -> lower=-0.8 upper=0.8 effort=1000.0 velocity=1000.0
